Commit message: smach manipulation

File: moveit_apps/urdf/table.urdf.xacro (robot description, xacro)
@@ -22,5 +22,5 @@
         <parent link="world" />
         <child link="table" />
-        <origin xyz="0.5 -0.25 0.75" rpy="0 0 0" />
+        <origin xyz="0.75 0.0 0.75" rpy="0 0 0" />
     </joint>
     <gazebo reference="table">

Commit message: added willowgarage map

File: moveit_apps/urdf/table.urdf.xacro (robot description, xacro)
@@ -9,10 +9,10 @@
         <visual>
             <geometry>
-                <box size="0.4 0.5 0.1"/>
+                <box size="0.4 0.5 0.75"/>
             </geometry>
         </visual>
         <collision>
             <geometry>
-                <box size="0.4 0.5 0.1"/>
+                <box size="0.4 0.5 0.75"/>
             </geometry>
         </collision>
@@ -22,5 +22,5 @@
         <parent link="world" />
         <child link="table" />
-        <origin xyz="0.75 0.0 0.75" rpy="0 0 0" />
+        <origin xyz="0.75 0.0 0.375" rpy="0 0 0" />
     </joint>
     <gazebo reference="table">
